Commit message: Added venv, updated kinematics.

File: basic_arm_modeling/arm.urdf (robot description, URDF)
Before this commit: robot simple_arm, 4 links, 3 joints
Links:
- added link hand; visual box size=0.1 0.05 0.05
- added link wrist; visual cylinder length=0.1 radius=0.03
- link arm1: geometry visual cylinder length=0.5 radius=0.05
- link arm2: geometry visual cylinder length=0.5 radius=0.05
Joints:
- added joint hand_joint: type revolute, parent wrist, child hand, origin xyz=0.0 0.0 0.1 rpy=0.0 0.0 0.0, axis 0.0 0.0 1.0, limit lower=-3.0 upper=3.0 effort=1000.0 velocity=1000.0
- added joint wrist_joint: type revolute, parent arm2, child wrist, origin xyz=0.0 0.0 0.5 rpy=0.0 0.0 0.0, axis 1.0 0.0 0.0, limit lower=-3.0 upper=3.0 effort=1000.0 velocity=1000.0
- joint arm1_joint: origin xyz=0.0 0.0 0.0 rpy=0.0 0.0 0.0 -> xyz=0.0 0.0 0.1 rpy=0.0 0.0 0.0
